File: esp-prog-adapter.kicad_pcb (KiCad board)
At the start: 2 copper layers, 25.4 x 21 mm, 4 parts, among them J1 ESP-PROG-Program, J2 ESP-PROG-Debug, J3 Conn_01x05_Male, J4 Conn_01x05_Male

Commit message: PCB layout changes
Parts:
- moved J3 0.63 mm to (82.5, 81.9)
- moved J4 0.63 mm to (74.9, 81.9)
Routing:
- net GND: track 4.91 -> 0.00 mm, vias 3 -> 2
- net /TDO: track 19.2 -> 19.8 mm
- net /EN: track 17.2 -> 17.8 mm
- net /TXD: track 19.3 -> 19.9 mm
- net /TMS: track 10.6 -> 11.2 mm
- net /TDI: track 24.1 -> 24.8 mm
- net /TCK: track 8.61 -> 9.25 mm
- net /RXD: track 20.6 -> 21.3 mm
- net /IO0: track 8.19 -> 8.83 mm
Other:
- board size 25.4 x 21 mm -> 25.4 x 22.2 mm

Commit message: Move ESP-PROG connectors to project library
Parts:
- J1: value ESP-PROG-Program -> Male IDC connector, 2x03, 1.27mm, SMD
- J2: value ESP-PROG-Debug -> Male IDC connector 2x05, 1.27mm, SMD
- J3, J4: value Conn_01x05_Male -> Pin header 1x05, 2.54mm
Changed lines of the file:
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@@
     (add_net /TXD)
     (add_net GND)
+    (add_net "Net-(J2-Pad10)")
     (add_net VCC)
   )
@@
       (effects (font (size 0.5 0.5) (thickness 0.125)) (justify right mirror))
     )
-    (fp_text value Conn_01x05_Male (at 11.43 -6.35 270) (layer B.Fab)
+    (fp_text value "Pin header 1x05, 2.54mm" (at 11.43 -6.35 270) (layer B.Fab)
       (effects (font (size 1 1) (thickness 0.15)))
     )
@@
       (effects (font (size 0.5 0.5) (thickness 0.125)) (justify left mirror))
     )
-    (fp_text value Conn_01x05_Male (at -11.43 -6.35 270) (layer B.Fab)
+    (fp_text value "Pin header 1x05, 2.54mm" (at -11.43 -6.35 270) (layer B.Fab)
       (effects (font (size 1 1) (thickness 0.15)))
     )
@@
       (effects (font (size 0.5 0.5) (thickness 0.125)) (justify left))
     )
-    (fp_text value ESP-PROG-Debug (at -4.445 3.81 180) (layer F.Fab)
+    (fp_text value "Male IDC connector 2x05, 1.27mm, SMD" (at -4.445 3.81 180) (layer F.Fab)
       (effects (font (size 1 1) (thickness 0.15)))
     )
@@
       (effects (font (size 0.5 0.5) (thickness 0.125)) (justify right))
     )
-    (fp_text value ESP-PROG-Program (at -4.445 -1.905 180) (layer F.Fab)
+    (fp_text value "Male IDC connector, 2x03, 1.27mm, SMD" (at -4.445 -1.905 180) (layer F.Fab)
       (effects (font (size 1 1) (thickness 0.15)))
     )
