File: modules/esp-32-board/esp-32-board.sch (KiCad schematic (older format))
At the start: 14 parts, among them J1 ESP-PROG-Program, J2 MainConnector, J3 ESP-PROG-Debug, J4 Conn_01x06, SW1 SW_Push, SW2 SW_Push, U1 ESP32-WROOM-32

Commit message: Replace MainConnector with ArduinoFootprint and separate headers
Parts:
- added J1: Conn_01x14_Female, Connector_PinSocket_2.54mm:PinSocket_1x14_P2.54mm_Vertical, symbol Connector:Conn_01x14_Female
- added J2: Conn_01x18_Female, Connector_PinSocket_2.54mm:PinSocket_1x18_P2.54mm_Vertical, symbol Connector:Conn_01x18_Female
- N1: renamed from J2; symbol project_components:MainConnector -> Mechanical:Housing
- renumbered J4 to J3, J1 to J6, J3 to J7
Connections:
- net +3V3: now also J1.1 (Pin_1), J2.18 (Pin_18); no longer N1.1 (Pin_1), N1.15 (Pin_15)
- net +5V: now also J2.1 (Pin_1); no longer N1.32 (Pin_32)
- net EN: now also J2.17 (Pin_17); no longer N1.16 (Pin_16)
- net GND: now also J1.14 (Pin_14), J2.2 (Pin_2); no longer N1.14 (Pin_14), N1.31 (Pin_31)
- net IO0: now also J1.2 (Pin_2); no longer N1.2 (Pin_2)
- net IO12: now also J2.6 (Pin_6); no longer N1.27 (Pin_27)
- net IO13: now also J2.5 (Pin_5); no longer N1.28 (Pin_28)
- net IO14: now also J2.7 (Pin_7); no longer N1.26 (Pin_26)
- net IO15: now also J2.4 (Pin_4); no longer N1.29 (Pin_29)
- net IO16: now also J1.4 (Pin_4); no longer N1.4 (Pin_4)
- net IO17: now also J1.5 (Pin_5); no longer N1.5 (Pin_5)
- net IO18: now also J1.7 (Pin_7); no longer N1.7 (Pin_7)
- net IO19: now also J1.8 (Pin_8); no longer N1.8 (Pin_8)
- net IO2: now also J2.3 (Pin_3); no longer N1.30 (Pin_30)
- net IO21: now also J1.9 (Pin_9); no longer N1.9 (Pin_9)
- net IO22: now also J1.12 (Pin_12); no longer N1.12 (Pin_12)
- net IO23: now also J1.13 (Pin_13); no longer N1.13 (Pin_13)
- net IO25: now also J2.10 (Pin_10); no longer N1.23 (Pin_23)
- net IO26: now also J2.9 (Pin_9); no longer N1.24 (Pin_24)
- net IO27: now also J2.8 (Pin_8); no longer N1.25 (Pin_25)
- net IO32: now also J2.12 (Pin_12); no longer N1.21 (Pin_21)
- net IO33: now also J2.11 (Pin_11); no longer N1.22 (Pin_22)
- net IO34: now also J2.14 (Pin_14); no longer N1.19 (Pin_19)
- net IO35: now also J2.13 (Pin_13); no longer N1.20 (Pin_20)
- net IO36: now also J2.16 (Pin_16); no longer N1.17 (Pin_17)
- net IO39: now also J2.15 (Pin_15); no longer N1.18 (Pin_18)
- net IO4: now also J1.3 (Pin_3); no longer N1.3 (Pin_3)
- net IO5: now also J1.6 (Pin_6); no longer N1.6 (Pin_6)
- net RXD0: now also J1.10 (Pin_10); no longer N1.10 (Pin_10)
- net TXD0: now also J1.11 (Pin_11); no longer N1.11 (Pin_11)
Changed lines of the file:
@@
 	7400 2400 6850 2400
 $Comp
-L Connector:ESP-PROG-Program J1
+L Connector:ESP-PROG-Program J6
 U 1 1 5FECB5F0
 P 7100 5600
-F 0 "J1" H 6750 6150 50  0000 L CNN
+F 0 "J6" H 6750 6150 50  0000 L CNN
 F 1 "ESP-PROG-Program" H 7250 6150 50  0000 L CNN
 F 2 "Connector_IDC:IDC-Header_2x03_P1.27mm_Vertical_SMD" V 6850 5650 50  0001 C CNN
@@
 	7100 6200 7100 6300
 $Comp
-L Connector:ESP-PROG-Debug J3
+L Connector:ESP-PROG-Debug J7
 U 1 1 5FF13734
 P 9100 5600
-F 0 "J3" H 8800 6150 50  0000 R CNN
+F 0 "J7" H 8800 6150 50  0000 R CNN
 F 1 "ESP-PROG-Debug" H 9850 6150 50  0000 R CNN
 F 2 "Connector_IDC:IDC-Header_2x05_P1.27mm_Vertical_SMD" V 8850 5650 50  0001 C CNN
@@
 	9500 5500 9800 5500
 $Comp
-L project_components:MainConnector J2
+L Mechanical:Housing N1
 U 1 1 600797C7
-P 7800 2550
-F 0 "J2" H 7800 3700 50  0000 C CNN
-F 1 "MainConnector" H 7800 3600 50  0000 C CNN
-F 2 "project_components:MainConnector" H 7600 2050 50  0001 C CNN
-F 3 "~" H 7600 2050 50  0001 C CNN
-F 4 "N/A" H 7800 2550 50  0001 C CNN "Vendor"
-	1    7800 2550
+P 6400 7400
+F 0 "N1" H 6400 7750 50  0000 C CNN
+F 1 "MainConnector" H 6400 7650 50  0000 C CNN
+F 2 "project_components:MainConnector" H 6200 6900 50  0001 C CNN
+F 3 "~" H 6200 6900 50  0001 C CNN
+F 4 "N/A" H 6400 7400 50  0001 C CNN "Vendor"
+	1    6400 7400
 	1    0    0    -1
 $EndComp
@@
 	6700 2000 7400 2000
 $Comp
-L Connector_Generic:Conn_01x06 J4
+L Connector_Generic:Conn_01x06 J3
 U 1 1 602A25F3
 P 10000 2450
-F 0 "J4" H 10000 2800 50  0000 C CNN
+F 0 "J3" H 10000 2800 50  0000 C CNN
 F 1 "Conn_01x06" H 10000 2000 50  0000 C CNN
 F 2 "Connector_PinSocket_2.54mm:PinSocket_1x06_P2.54mm_Vertical" H 10000 2450 50  0001 C CNN
@@
 Wire Wire Line
 	5150 3000 5500 3000
+$Comp
+L Connector:Conn_01x14_Female J1
+U 1 1 60EBE89E
+P 7600 2600
+F 0 "J1" H 7250 3650 50  0000 C CNN
+F 1 "Conn_01x14_Female" H 7300 3550 50  0000 C CNN
+F 2 "Connector_PinSocket_2.54mm:PinSocket_1x14_P2.54mm_Vertical" H 7600 2600 50  0001 C CNN
+F 3 "~" H 7600 2600 50  0001 C CNN
+	1    7600 2600
+	1    0    0    -1
+$EndComp
+$Comp
+L Connector:Conn_01x18_Female J2
+U 1 1 60ECF59A
+P 8000 2550
+F 0 "J2" H 7850 3550 50  0000 C CNN
+F 1 "Conn_01x18_Female" H 7850 3450 50  0000 C CNN
+F 2 "Connector_PinSocket_2.54mm:PinSocket_1x18_P2.54mm_Vertical" H 8000 2550 50  0001 C CNN
+F 3 "~" H 8000 2550 50  0001 C CNN
+	1    8000 2550
+	-1   0    0    -1
+$EndComp
 $EndSCHEMATC

Commit message: Add custom symbols/footprints to project_components
Parts:
- J6: footprint Connector_IDC:IDC-Header_2x03_P1.27mm_Vertical_SMD -> project_components:IDC-Header_2x03_P1.27mm_Vertical_SMD; symbol Connector:ESP-PROG-Program -> project_components:ESP-PROG-Program
- J7: footprint Connector_IDC:IDC-Header_2x05_P1.27mm_Vertical_SMD -> project_components:IDC-Header_2x05_P1.27mm_Vertical_SMD; symbol Connector:ESP-PROG-Debug -> project_components:ESP-PROG-Debug
- N1: value MainConnector -> Arduino Footprint; footprint project_components:MainConnector -> project_components:ArduinoFootprint
- SW1, SW2: footprint Button_Switch_SMD:SW_Push_1P1T_NO_6x6mm_H4.3mm -> project_components:SW_Push_1P1T_NO_6x6mm_H4.3mm
- U1: footprint RF_Module:ESP32-WROOM-32-ThermalVias -> project_components:ESP32-WROOM-32-ThermalVias
Changed lines of the file:
@@
 F 0 "U1" H 1600 4400 50  0000 C CNN
 F 1 "ESP32-WROOM-32" H 2700 4400 50  0000 C CNN
-F 2 "RF_Module:ESP32-WROOM-32-ThermalVias" H 2100 1500 50  0000 C CNN
+F 2 "project_components:ESP32-WROOM-32-ThermalVias" H 2100 1500 50  0000 C CNN
 F 3 "https://www.espressif.com/sites/default/files/documentation/esp32-wroom-32_datasheet_en.pdf" H 1800 3050 50  0001 C CNN
 	1    2100 3000
@@
 F 0 "SW1" H 4850 3250 50  0000 C CNN
 F 1 "SW_Push" H 4850 3150 50  0000 C CNN
-F 2 "Button_Switch_SMD:SW_Push_1P1T_NO_6x6mm_H4.3mm" H 4850 3200 50  0001 C CNN
+F 2 "project_components:SW_Push_1P1T_NO_6x6mm_H4.3mm" H 4850 3200 50  0001 C CNN
 F 3 "" H 4850 3200 50  0001 C CNN
 F 4 "tme.eu" H 4850 3000 50  0001 C CNN "Vendor"
@@
 F 0 "SW2" H 4850 4600 50  0000 C CNN
 F 1 "SW_Push" H 4850 4500 50  0000 C CNN
-F 2 "Button_Switch_SMD:SW_Push_1P1T_NO_6x6mm_H4.3mm" H 4850 4500 50  0001 C CNN
+F 2 "project_components:SW_Push_1P1T_NO_6x6mm_H4.3mm" H 4850 4500 50  0001 C CNN
 F 3 "" H 4850 4500 50  0001 C CNN
 F 4 "tme.eu" H 4850 4300 50  0001 C CNN "Vendor"
@@
 	7400 2400 6850 2400
 $Comp
-L Connector:ESP-PROG-Program J6
+L project_components:ESP-PROG-Program J6
 U 1 1 5FECB5F0
 P 7100 5600
 F 0 "J6" H 6750 6150 50  0000 L CNN
 F 1 "ESP-PROG-Program" H 7250 6150 50  0000 L CNN
-F 2 "Connector_IDC:IDC-Header_2x03_P1.27mm_Vertical_SMD" V 6850 5650 50  0001 C CNN
+F 2 "project_components:IDC-Header_2x03_P1.27mm_Vertical_SMD" V 6850 5650 50  0001 C CNN
 F 3 "https://github.com/espressif/esp-iot-solution/blob/master/documents/evaluation_boards/ESP-Prog_guide_en.md" H 5825 5050 50  0001 C CNN
 F 4 "https://www.ebay.com/itm/10Pcs-1-27mm-Pitch-2x3-Pin-6-Pin-SMT-SMD-Male-Shrouded-Box-Header-IDC-Connector/183523538792?hash=item2abadaf768:g:-H4AAOSwm-Fb4s52" H 7100 5600 50  0001 C CNN "VendorLink"
@@
 	7100 6200 7100 6300
 $Comp
-L Connector:ESP-PROG-Debug J7
+L project_components:ESP-PROG-Debug J7
 U 1 1 5FF13734
 P 9100 5600
 F 0 "J7" H 8800 6150 50  0000 R CNN
 F 1 "ESP-PROG-Debug" H 9850 6150 50  0000 R CNN
-F 2 "Connector_IDC:IDC-Header_2x05_P1.27mm_Vertical_SMD" V 8850 5650 50  0001 C CNN
+F 2 "project_components:IDC-Header_2x05_P1.27mm_Vertical_SMD" V 8850 5650 50  0001 C CNN
 F 3 "https://github.com/espressif/esp-iot-solution/blob/master/documents/evaluation_boards/ESP-Prog_guide_en.md" H 7825 5050 50  0001 C CNN
 F 4 "https://www.ebay.com/itm/5Pcs-1-27mm-Pitch-2x5-Pin-10-Pin-SMT-SMD-Male-Shrouded-Box-Header-IDC-Connector/172311876086?hash=item281e9691f6:g:eHIAAOSwu6taWHc7" H 9100 5600 50  0001 C CNN "VendorLink"
@@
 P 6400 7400
 F 0 "N1" H 6400 7750 50  0000 C CNN
-F 1 "MainConnector" H 6400 7650 50  0000 C CNN
-F 2 "project_components:MainConnector" H 6200 6900 50  0001 C CNN
+F 1 "Arduino Footprint" H 6400 7650 50  0000 C CNN
+F 2 "project_components:ArduinoFootprint" H 6200 6900 50  0001 C CNN
 F 3 "~" H 6200 6900 50  0001 C CNN
 F 4 "N/A" H 6400 7400 50  0001 C CNN "Vendor"

Commit message: Documentational changes
Connections:
- net TMS': now reaches J7.2 (ESP_TMS), RN1.4 (R4.1)
- net TCK': now reaches J7.4 (ESP_TCK), RN1.3 (R3.1)
- net TDO': now reaches J7.6 (ESP_TDO), RN1.2 (R2.1)
- net TDI': now reaches J7.8 (ESP_TDI), RN1.1 (R1.1)
Other:
- note added: "* from ESP-WROOM-32 datasheet:\n\nPins SCK/CLK, SDO/SD0, SDI/SD1,\nSHD/SD2, SWP/SD3 and SCS/CMD,\nnamely, GPIO6 to GPIO11 are\nconnected to the integrated SPI flash\nintegrated on the module and\nare not recommended for other uses."
- note added: "Buttons"
- note added: "Footprint"
- note added: "Power"
- note added: "Source: https://docs.espressif.com/projects/espressif-esp-iot-solution/en/latest/hw-reference/ESP-Prog_guide.html"
- note added: "USB"
- note removed: "Power & USB"
- moved on the sheet: C1, C2, C3, C4, J1, J2, J3, J6, J7, R5, R6, RN1A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
