File: modules/power-meter-hat/power_channel.kicad_sch (KiCad schematic)
At the start: 8 parts, among them J5 OutputTerminal, U5 INA219AxD

Commit message: Change jumpers
Parts:
- removed J5: OutputTerminal, TerminalBlock_Phoenix:TerminalBlock_Phoenix_PT-1,5-2-3.5-H_1x02_P3.50mm_Horizontal, symbol Connector_Generic:Conn_01x02
- removed JP10: Jumper, Connector_PinHeader_2.54mm:PinHeader_1x03_P2.54mm_Vertical, symbol Jumper:Jumper_3_Open
- added J3: OutputTerminal, TerminalBlock_Phoenix:TerminalBlock_Phoenix_PT-1,5-4-3.5-H_1x04_P3.50mm_Horizontal, symbol Connector_Generic:Conn_01x04
- renumbered D5 to D3, JP9 to JP3, JP11 to JP4, R14 to R10, R13 to R9, U5 to U3
Connections:
- net GND: now also J3.2 (Pin_2), J3.4 (Pin_4)
- net IN_VCC renamed VIN
- net VIN: now also JP3.2 (C); no longer JP3.1 (A)
- net OUT_VCC renamed VOUT
- net VOUT: now also J3.3 (Pin_3)
- net PWR renamed INTERNAL_VIN
- net INTERNAL_VIN: no longer JP3.2 (C)
- new net EXTERNAL_VIN: J3.1 (Pin_1), JP3.1 (A)

Commit message: Add bypass capacitors for INA219
Parts:
- added C4: 100n, Capacitor_SMD:C_0805_2012Metric_Pad1.18x1.45mm_HandSolder, symbol Device:C
Connections:
- net +3.3V: now also C4.1
- net GND: now also C4.2
Changed lines of the file:
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@@
   (junction (at 139.7 29.21) (diameter 0) (color 0 0 0 0)
   )
+  (junction (at 128.27 87.63) (diameter 0) (color 0 0 0 0)
+  )
+  (junction (at 128.27 64.77) (diameter 0) (color 0 0 0 0)
+  )
   (junction (at 113.665 69.85) (diameter 0) (color 0 0 0 0)
   )
+  (wire (pts (xy 128.27 87.63) (xy 157.48 87.63))
+    (stroke (width 0) (type default) (color 0 0 0 0))
+  )
   (wire (pts (xy 146.685 24.13) (xy 139.7 24.13))
     (stroke (width 0) (type default) (color 0 0 0 0))
@@
     (stroke (width 0) (type default) (color 0 0 0 0))
   )
+  (wire (pts (xy 157.48 87.63) (xy 157.48 80.01))
+    (stroke (width 0) (type default) (color 0 0 0 0))
+  )
   (wire (pts (xy 117.475 69.85) (xy 117.475 73.66))
     (stroke (width 0) (type default) (color 0 0 0 0))
@@
     (stroke (width 0) (type default) (color 0 0 0 0))
   )
-  (wire (pts (xy 128.27 63.5) (xy 128.27 66.04))
+  (wire (pts (xy 128.27 63.5) (xy 128.27 64.77))
     (stroke (width 0) (type default) (color 0 0 0 0))
   )
@@
     (stroke (width 0) (type default) (color 0 0 0 0))
   )
+  (wire (pts (xy 128.27 64.77) (xy 128.27 66.04))
+    (stroke (width 0) (type default) (color 0 0 0 0))
+  )
   (wire (pts (xy 101.6 69.85) (xy 113.665 69.85))
     (stroke (width 0) (type default) (color 0 0 0 0))
   )
+  (wire (pts (xy 128.27 87.63) (xy 128.27 88.9))
+    (stroke (width 0) (type default) (color 0 0 0 0))
+  )
   (wire (pts (xy 123.825 26.67) (xy 146.685 26.67))
     (stroke (width 0) (type default) (color 0 0 0 0))
@@
     (stroke (width 0) (type default) (color 0 0 0 0))
   )
-  (wire (pts (xy 128.27 86.36) (xy 128.27 88.9))
+  (wire (pts (xy 128.27 86.36) (xy 128.27 87.63))
+    (stroke (width 0) (type default) (color 0 0 0 0))
+  )
+  (wire (pts (xy 128.27 64.77) (xy 157.48 64.77))
     (stroke (width 0) (type default) (color 0 0 0 0))
   )
@@
   )
   (wire (pts (xy 138.43 78.74) (xy 146.05 78.74))
+    (stroke (width 0) (type default) (color 0 0 0 0))
+  )
+  (wire (pts (xy 157.48 64.77) (xy 157.48 72.39))
     (stroke (width 0) (type default) (color 0 0 0 0))
   )
@@
     (pin "3")
   )
+  (symbol (lib_id "Device:C") (at 157.48 76.2 0)
+    (in_bom yes) (on_board yes) (fields_autoplaced)
+    (property "Reference" "C4" (id 0) (at 161.29 74.9299 0)
+      (effects (font (size 1.27 1.27)) (justify left))
+    )
+    (property "Value" "100n" (id 1) (at 161.29 77.4699 0)
+      (effects (font (size 1.27 1.27)) (justify left))
+    )
+    (property "Footprint" "Capacitor_SMD:C_0805_2012Metric_Pad1.18x1.45mm_HandSolder" (id 2) (at 158.4452 80.01 0)
+      (effects (font (size 1.27 1.27)) hide)
+    )
+    (property "Datasheet" "~" (id 3) (at 157.48 76.2 0)
+      (effects (font (size 1.27 1.27)) hide)
+    )
+    (pin "1")
+    (pin "2")
+  )
   (symbol (lib_id "power:+3.3V") (at 128.27 63.5 0)
     (in_bom yes) (on_board yes) (fields_autoplaced)
-    (property "Reference" "#PWR039" (id 0) (at 128.27 67.31 0)
+    (property "Reference" "#PWR024" (id 0) (at 128.27 67.31 0)
       (effects (font (size 1.27 1.27)) hide)
     )
@@
   (symbol (lib_id "power:GND") (at 184.15 60.96 0)
     (in_bom yes) (on_board yes) (fields_autoplaced)
-    (property "Reference" "#PWR043" (id 0) (at 184.15 67.31 0)
+    (property "Reference" "#PWR027" (id 0) (at 184.15 67.31 0)
       (effects (font (size 1.27 1.27)) hide)
     )
@@
   (symbol (lib_id "power:+3.3VP") (at 76.2 25.4 0)
     (in_bom yes) (on_board yes) (fields_autoplaced)
-    (property "Reference" "#PWR037" (id 0) (at 80.01 26.67 0)
+    (property "Reference" "#PWR022" (id 0) (at 80.01 26.67 0)
       (effects (font (size 1.27 1.27)) hide)
     )
@@
   (symbol (lib_id "power:+5VP") (at 101.6 25.4 0)
     (in_bom yes) (on_board yes) (fields_autoplaced)
-    (property "Reference" "#PWR038" (id 0) (at 101.6 29.21 0)
+    (property "Reference" "#PWR023" (id 0) (at 101.6 29.21 0)
       (effects (font (size 1.27 1.27)) hide)
     )
@@
   (symbol (lib_id "power:GND") (at 128.27 88.9 0)
     (in_bom yes) (on_board yes) (fields_autoplaced)
-    (property "Reference" "#PWR040" (id 0) (at 128.27 95.25 0)
+    (property "Reference" "#PWR025" (id 0) (at 128.27 95.25 0)
       (effects (font (size 1.27 1.27)) hide)
     )
@@
   (symbol (lib_id "power:GND") (at 139.7 34.29 0)
     (in_bom yes) (on_board yes) (fields_autoplaced)
-    (property "Reference" "#PWR041" (id 0) (at 139.7 40.64 0)
-      (effects (font (size 1.27 1.27)) hide)
-    )
+    (property "Reference" "#PWR026" (id 0) (at 139.7 40.64 0)
+      (effects (font (size 1.27 1.27)) hide)
+    )
