File: modules/power-monitor-hat/power-monitor-hat.kicad_sch (KiCad schematic)
At the start: 25 parts, among them J1 Barrel_Jack_Switch, J2 GPIO, Q1 BC856BDW1, Q2 SI2301CDS, U1 CAT24C256, U2 NCP1117-3.3_SOT223

Commit message: Add separate net for "power ground"
Parts:
- renumbered R5 to R3, R6 to R4, R4 to R5, R3 to R6, U2 to U1, U1 to U2
Connections:
- net GND: no longer C2.2, C3.2, J1.2, J1.3, J2.25 (GND), R1.2, R2.2, U1.1 (GND)
- new net GNDPWR: C2.2, C3.2, J1.2, J1.3, J2.25 (GND), R1.2, R2.2, U1.1 (GND)
Other:
- moved on the sheet: R5, R6

Commit message: Correct units
Parts:
- C2, C3: value 22u -> 10u
- R3, R4: value 220R -> 470R
- TP1, TP2, TP3: footprint TestPoint:TestPoint_Loop_D2.54mm_Drill1.5mm_Beaded -> TestPoint:TestPoint_Loop_D1.80mm_Drill1.0mm_Beaded
Changed lines of the file:
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@@
       (effects (font (size 1.27 1.27)) (justify left))
     )
-    (property "Value" "22u" (id 1) (at 137.16 135.2549 0)
+    (property "Value" "10u" (id 1) (at 137.16 135.2549 0)
       (effects (font (size 1.27 1.27)) (justify left))
     )
@@
       (effects (font (size 1.27 1.27)) (justify left))
     )
-    (property "Value" "22u" (id 1) (at 162.56 135.2549 0)
+    (property "Value" "10u" (id 1) (at 162.56 135.2549 0)
       (effects (font (size 1.27 1.27)) (justify left))
     )
@@
       (effects (font (size 1.27 1.27)) (justify left))
     )
-    (property "Footprint" "TestPoint:TestPoint_Loop_D2.54mm_Drill1.5mm_Beaded" (id 2) (at 144.78 177.8 0)
+    (property "Footprint" "TestPoint:TestPoint_Loop_D1.80mm_Drill1.0mm_Beaded" (id 2) (at 144.78 177.8 0)
       (effects (font (size 1.27 1.27)) hide)
     )
@@
     (in_bom yes) (on_board yes)
     (property "Reference" "R4" (id 0) (at 141.224 50.038 0))
-    (property "Value" "220R" (id 1) (at 141.224 52.578 0))
+    (property "Value" "470R" (id 1) (at 141.224 52.578 0))
     (property "Footprint" "Resistor_SMD:R_0805_2012Metric_Pad1.20x1.40mm_HandSolder" (id 2) (at 146.812 50.038 90)
       (effects (font (size 1.27 1.27)) hide)
@@
       (effects (font (size 1.27 1.27)) (justify left))
     )
-    (property "Footprint" "TestPoint:TestPoint_Loop_D2.54mm_Drill1.5mm_Beaded" (id 2) (at 157.48 177.8 0)
+    (property "Footprint" "TestPoint:TestPoint_Loop_D1.80mm_Drill1.0mm_Beaded" (id 2) (at 157.48 177.8 0)
       (effects (font (size 1.27 1.27)) hide)
     )
@@
       (effects (font (size 1.27 1.27)) (justify left))
     )
-    (property "Footprint" "TestPoint:TestPoint_Loop_D2.54mm_Drill1.5mm_Beaded" (id 2) (at 132.08 177.8 0)
+    (property "Footprint" "TestPoint:TestPoint_Loop_D1.80mm_Drill1.0mm_Beaded" (id 2) (at 132.08 177.8 0)
       (effects (font (size 1.27 1.27)) hide)
     )
@@
     (in_bom yes) (on_board yes)
     (property "Reference" "R3" (id 0) (at 128.27 48.895 0))
-    (property "Value" "220R" (id 1) (at 127.635 51.435 0))
+    (property "Value" "470R" (id 1) (at 127.635 51.435 0))
     (property "Footprint" "Resistor_SMD:R_0805_2012Metric_Pad1.20x1.40mm_HandSolder" (id 2) (at 133.858 49.53 90)
       (effects (font (size 1.27 1.27)) hide)
@@
     )
     (path "/03e6e53e-2294-4c17-8562-f1d13ac7052a"
-      (reference "C2") (unit 1) (value "22u") (footprint "Capacitor_SMD:C_0805_2012Metric_Pad1.18x1.45mm_HandSolder")
+      (reference "C2") (unit 1) (value "10u") (footprint "Capacitor_SMD:C_0805_2012Metric_Pad1.18x1.45mm_HandSolder")
     )
     (path "/0defe58a-c9b1-4a12-9196-1eca934131ff"
-      (reference "C3") (unit 1) (value "22u") (footprint "Capacitor_SMD:C_0805_2012Metric_Pad1.18x1.45mm_HandSolder")
+      (reference "C3") (unit 1) (value "10u") (footprint "Capacitor_SMD:C_0805_2012Metric_Pad1.18x1.45mm_HandSolder")
     )
     (path "/7acdcd65-592b-4fae-a99e-c444a4b4e6be/1763cfc1-ab16-4cc7-8cff-020d06797821"
@@
     )
     (path "/fb8a5447-fc31-4f17-800d-6b1f88a9811b"
-      (reference "R3") (unit 1) (value "220R") (footprint "Resistor_SMD:R_0805_2012Metric_Pad1.20x1.40mm_HandSolder")
+      (reference "R3") (unit 1) (value "470R") (footprint "Resistor_SMD:R_0805_2012Metric_Pad1.20x1.40mm_HandSolder")
     )
     (path "/3ebe71a8-33cd-4a83-abc8-b064b502ad7a"
-      (reference "R4") (unit 1) (value "220R") (footprint "Resistor_SMD:R_0805_2012Metric_Pad1.20x1.40mm_HandSolder")
+      (reference "R4") (unit 1) (value "470R") (footprint "Resistor_SMD:R_0805_2012Metric_Pad1.20x1.40mm_HandSolder")
     )
     (path "/510c400a-2410-46b0-a7fb-1072fc4f848b"
@@
     )
     (path "/7acdcd65-592b-4fae-a99e-c444a4b4e6be/3328ecae-0710-4f87-b7ab-e1ff877ecfd0"
-      (reference "R10") (unit 1) (value "220R") (footprint "Resistor_SMD:R_0805_2012Metric_Pad1.20x1.40mm_HandSolder")
+      (reference "R10") (unit 1) (value "470R") (footprint "Resistor_SMD:R_0805_2012Metric_Pad1.20x1.40mm_HandSolder")
     )
     (path "/5773e18f-350c-4982-8a03-ea7374ba7702/1e56e336-29d0-480b-b322-a3d599057f32"
@@
     )
     (path "/5773e18f-350c-4982-8a03-ea7374ba7702/3328ecae-0710-4f87-b7ab-e1ff877ecfd0"
-      (reference "R12") (unit 1) (value "220R") (footprint "Resistor_SMD:R_0805_2012Metric_Pad1.20x1.40mm_HandSolder")
+      (reference "R12") (unit 1) (value "470R") (footprint "Resistor_SMD:R_0805_2012Metric_Pad1.20x1.40mm_HandSolder")
     )
     (path "/19fa45c1-8471-4c12-ac70-3f183c159f90/1e56e336-29d0-480b-b322-a3d599057f32"
@@
     )
     (path "/19fa45c1-8471-4c12-ac70-3f183c159f90/3328ecae-0710-4f87-b7ab-e1ff877ecfd0"
-      (reference "R14") (unit 1) (value "220R") (footprint "Resistor_SMD:R_0805_2012Metric_Pad1.20x1.40mm_HandSolder")
+      (reference "R14") (unit 1) (value "470R") (footprint "Resistor_SMD:R_0805_2012Metric_Pad1.20x1.40mm_HandSolder")
     )
     (path "/ea0ee2c9-885b-4c4e-992a-86782e1a690a"
-      (reference "TP1") (unit 1) (value "TestPoint") (footprint "TestPoint:TestPoint_Loop_D2.54mm_Drill1.5mm_Beaded")
+      (reference "TP1") (unit 1) (value "TestPoint") (footprint "TestPoint:TestPoint_Loop_D1.80mm_Drill1.0mm_Beaded")
     )
     (path "/359d4095-7e08-4e54-945e-63f380a9ecd6"
-      (reference "TP2") (unit 1) (value "TestPoint") (footprint "TestPoint:TestPoint_Loop_D2.54mm_Drill1.5mm_Beaded")
+      (reference "TP2") (unit 1) (value "TestPoint") (footprint "TestPoint:TestPoint_Loop_D1.80mm_Drill1.0mm_Beaded")
     )
     (path "/b9e161cf-bac5-49df-96d6-921605a35e99"
-      (reference "TP3") (unit 1) (value "TestPoint") (footprint "TestPoint:TestPoint_Loop_D2.54mm_Drill1.5mm_Beaded")
+      (reference "TP3") (unit 1) (value "TestPoint") (footprint "TestPoint:TestPoint_Loop_D1.80mm_Drill1.0mm_Beaded")
     )
     (path "/019b9904-3bfd-4fd4-9d41-96b38c16849e"

Commit message: Silkscreen improvement
Other:
- note removed: "Additional pin functions: https://pinout.xyz/"
- title: (none) -> ${DISPLAY_NAME}
Changed lines of the file:
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@@
   (paper "A4")
   (title_block
+    (title "${DISPLAY_NAME}")
     (date "15 nov 2012")
+    (rev "v${VERSION}")
+    (comment 1 "URL: ${URL}")
   )
   (junction (at 203.2 67.31) (diameter 0) (color 0 0 0 0)
@@
     (stroke (width 0) (type default) (color 0 0 0 0))
   )
-  (text "Additional pin functions:\nhttps://pinout.xyz/" (at 179.07 180.34 0)
-    (effects (font (size 1.27 1.27)) (justify left bottom))
-  )
   (text "+5V power circuit" (at 59.69 115.57 0)

Commit message: Remove top LED, connect channel LEDs to VIN, expose RX/TX header
Parts:
- removed D2: LED, LED_SMD:LED_1206_3216Metric, symbol Device:LED
- removed R4: 470R, Resistor_SMD:R_0805_2012Metric_Pad1.20x1.40mm_HandSolder, symbol Device:R
- added J6: Conn_01x03, Connector_PinHeader_2.54mm:PinHeader_1x03_P2.54mm_Vertical, symbol Connector_Generic:Conn_01x03
Connections:
- net GND: now also J6.1 (Pin_1)
- net RX: now reaches J2.10 (GPIO15/RXD)
- net RX: now also J6.2 (Pin_2)
- net TX: now reaches J2.8 (GPIO14/TXD)
- net TX: now also J6.3 (Pin_3)
- net LED: no longer names the net of J2.16 (GPIO23)
- net LED_CH1: no longer names the net of J2.11 (GPIO17)
- net LED_CH2: no longer names the net of J2.13 (GPIO27)
- net LED_CH3: no longer names the net of J2.15 (GPIO22)
- no-connect marks 23 -> 25
Other:
- sheet PowerChannel 1 ports: added none; removed LED
- sheet PowerChannel 2 ports: added none; removed LED
- sheet PowerChannel 3 ports: added none; removed LED
- note added: "Top LED"
- note removed: "Top LEDs"
- moved on the sheet: D1, R3, TP1, TP2, TP3
