File: modules/power-monitor-hat/power_channel.kicad_sch (KiCad schematic)
At the start: 8 parts, among them J3 OutputTerminal, U3 INA219AxD

Commit message: Add separate net for "power ground"
Connections:
- net GND: no longer J3.2 (Pin_2), J3.4 (Pin_4)
- new net GNDPWR: J3.2 (Pin_2), J3.4 (Pin_4)
Changed lines of the file:
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@@
   (symbol (lib_id "power:+3.3V") (at 128.27 63.5 0)
     (in_bom yes) (on_board yes) (fields_autoplaced)
-    (property "Reference" "#PWR024" (id 0) (at 128.27 67.31 0)
+    (property "Reference" "#PWR038" (id 0) (at 128.27 67.31 0)
       (effects (font (size 1.27 1.27)) hide)
     )
@@
   (symbol (lib_id "power:GND") (at 184.15 60.96 0)
     (in_bom yes) (on_board yes) (fields_autoplaced)
-    (property "Reference" "#PWR027" (id 0) (at 184.15 67.31 0)
+    (property "Reference" "#PWR041" (id 0) (at 184.15 67.31 0)
       (effects (font (size 1.27 1.27)) hide)
     )
@@
   (symbol (lib_id "power:+3.3VP") (at 76.2 25.4 0)
     (in_bom yes) (on_board yes) (fields_autoplaced)
-    (property "Reference" "#PWR022" (id 0) (at 80.01 26.67 0)
+    (property "Reference" "#PWR036" (id 0) (at 80.01 26.67 0)
       (effects (font (size 1.27 1.27)) hide)
     )
@@
   (symbol (lib_id "power:+5VP") (at 101.6 25.4 0)
     (in_bom yes) (on_board yes) (fields_autoplaced)
-    (property "Reference" "#PWR023" (id 0) (at 101.6 29.21 0)
+    (property "Reference" "#PWR037" (id 0) (at 101.6 29.21 0)
       (effects (font (size 1.27 1.27)) hide)
     )
@@
   (symbol (lib_id "power:GND") (at 128.27 88.9 0)
     (in_bom yes) (on_board yes) (fields_autoplaced)
-    (property "Reference" "#PWR025" (id 0) (at 128.27 95.25 0)
+    (property "Reference" "#PWR039" (id 0) (at 128.27 95.25 0)
       (effects (font (size 1.27 1.27)) hide)
     )
@@
     (pin "1")
   )
-  (symbol (lib_id "power:GND") (at 139.7 34.29 0)
+  (symbol (lib_id "power:GNDPWR") (at 139.7 34.29 0)
     (in_bom yes) (on_board yes) (fields_autoplaced)
-    (property "Reference" "#PWR026" (id 0) (at 139.7 40.64 0)
+    (property "Reference" "#PWR040" (id 0) (at 139.7 39.37 0)
       (effects (font (size 1.27 1.27)) hide)
     )
-    (property "Value" "GND" (id 1) (at 139.7 39.37 0))
-    (property "Footprint" "" (id 2) (at 139.7 34.29 0)
+    (property "Value" "GNDPWR" (id 1) (at 139.573 38.735 0))
+    (property "Footprint" "" (id 2) (at 139.7 35.56 0)
       (effects (font (size 1.27 1.27)) hide)
     )
-    (property "Datasheet" "" (id 3) (at 139.7 34.29 0)
+    (property "Datasheet" "" (id 3) (at 139.7 35.56 0)
       (effects (font (size 1.27 1.27)) hide)
     )

Commit message: Change footprint for jumpers to "no first pin" version
Parts:
- JP3, JP4: footprint Connector_PinHeader_2.54mm:PinHeader_1x03_P2.54mm_Vertical -> shared_components:PinHeader_1x03_P2.54mm_Vertical_NoFP
Connections:
- net +3.3VP: now also JP4.3 (B); no longer JP4.1 (A)
- net +5VP: now also JP4.1 (A); no longer JP4.3 (B)
Other:
- moved on the sheet: JP3

Commit message: Enhancements
Parts:
- R9: value R -> 0R5
Changed lines of the file:
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@@
       (effects (font (size 1.27 1.27)) (justify left))
     )
-    (property "Value" "R" (id 1) (at 115.57 77.4699 0)
+    (property "Value" "0R5" (id 1) (at 115.57 77.4699 0)
       (effects (font (size 1.27 1.27)) (justify left))
     )

Commit message: Correct units
Parts:
- R10: value 220R -> 470R
Changed lines of the file:
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@@
     (in_bom yes) (on_board yes) (fields_autoplaced)
     (property "Reference" "R10" (id 0) (at 177.8 52.07 90))
-    (property "Value" "220R" (id 1) (at 180.34 52.07 90))
+    (property "Value" "470R" (id 1) (at 180.34 52.07 90))
     (property "Footprint" "Resistor_SMD:R_0805_2012Metric_Pad1.20x1.40mm_HandSolder" (id 2) (at 185.928 52.07 90)
       (effects (font (size 1.27 1.27)) hide)

Commit message: Silkscreen improvement
Parts:
- renumbered C4 to C6, D3 to D5, J3 to J5, JP3 to JP7, JP4 to JP8, R9 to R13, R10 to R14, U3 to U5
Changed lines of the file:
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@@
   (symbol (lib_id "Jumper:Jumper_3_Open") (at 69.85 63.5 0)
     (in_bom yes) (on_board yes)
-    (property "Reference" "JP3" (id 0) (at 69.85 57.15 0))
+    (property "Reference" "JP7" (id 0) (at 69.85 57.15 0))
     (property "Value" "Jumper" (id 1) (at 62.23 67.31 0))
     (property "Footprint" "shared_components:PinHeader_1x03_P2.54mm_Vertical_NoFP" (id 2) (at 69.85 63.5 0)
@@
   (symbol (lib_id "Device:C") (at 157.48 76.2 0)
     (in_bom yes) (on_board yes) (fields_autoplaced)
-    (property "Reference" "C4" (id 0) (at 161.29 74.9299 0)
+    (property "Reference" "C6" (id 0) (at 161.29 74.9299 0)
       (effects (font (size 1.27 1.27)) (justify left))
     )
@@
   (symbol (lib_id "power:+3.3V") (at 128.27 63.5 0)
     (in_bom yes) (on_board yes) (fields_autoplaced)
-    (property "Reference" "#PWR026" (id 0) (at 128.27 67.31 0)
+    (property "Reference" "#PWR038" (id 0) (at 128.27 67.31 0)
       (effects (font (size 1.27 1.27)) hide)
     )
@@
   (symbol (lib_id "Device:R") (at 113.665 76.2 0)
     (in_bom yes) (on_board yes) (fields_autoplaced)
-    (property "Reference" "R9" (id 0) (at 115.57 74.9299 0)
+    (property "Reference" "R13" (id 0) (at 115.57 74.9299 0)
       (effects (font (size 1.27 1.27)) (justify left))
     )
@@
   (symbol (lib_id "Analog_ADC:INA219AxD") (at 128.27 76.2 0)
     (in_bom yes) (on_board yes) (fields_autoplaced)
-    (property "Reference" "U3" (id 0) (at 130.2894 63.5 0)
+    (property "Reference" "U5" (id 0) (at 130.2894 63.5 0)
       (effects (font (size 1.27 1.27)) (justify left))
     )
@@
   (symbol (lib_id "Device:R") (at 184.15 52.07 180)
     (in_bom yes) (on_board yes) (fields_autoplaced)
-    (property "Reference" "R10" (id 0) (at 177.8 52.07 90))
+    (property "Reference" "R14" (id 0) (at 177.8 52.07 90))
     (property "Value" "470R" (id 1) (at 180.34 52.07 90))
     (property "Footprint" "Resistor_SMD:R_0805_2012Metric_Pad1.20x1.40mm_HandSolder" (id 2) (at 185.928 52.07 90)
@@
   (symbol (lib_id "power:GND") (at 184.15 60.96 0)
     (in_bom yes) (on_board yes) (fields_autoplaced)
-    (property "Reference" "#PWR029" (id 0) (at 184.15 67.31 0)
+    (property "Reference" "#PWR041" (id 0) (at 184.15 67.31 0)
       (effects (font (size 1.27 1.27)) hide)
     )
@@
   (symbol (lib_id "Jumper:Jumper_3_Open") (at 88.9 31.75 0)
     (in_bom yes) (on_board yes)
-    (property "Reference" "JP4" (id 0) (at 88.9 25.4 0))
+    (property "Reference" "JP8" (id 0) (at 88.9 25.4 0))
     (property "Value" "Jumper" (id 1) (at 88.9 38.735 0))
     (property "Footprint" "shared_components:PinHeader_1x03_P2.54mm_Vertical_NoFP" (id 2) (at 88.9 31.75 0)
@@
   (symbol (lib_id "power:+3.3VP") (at 101.6 25.4 0) (mirror y)
     (in_bom yes) (on_board yes) (fields_autoplaced)
-    (property "Reference" "#PWR024" (id 0) (at 97.79 26.67 0)
+    (property "Reference" "#PWR036" (id 0) (at 97.79 26.67 0)
       (effects (font (size 1.27 1.27)) hide)
     )
@@
   (symbol (lib_id "Device:LED") (at 184.15 38.735 90)
     (in_bom yes) (on_board yes) (fields_autoplaced)
-    (property "Reference" "D3" (id 0) (at 191.77 40.3225 0))
+    (property "Reference" "D5" (id 0) (at 191.77 40.3225 0))
     (property "Value" "LED" (id 1) (at 189.23 40.3225 0))
     (property "Footprint" "LED_SMD:LED_1206_3216Metric" (id 2) (at 184.15 38.735 0)
@@
   (symbol (lib_id "Connector_Generic:Conn_01x04") (at 151.765 24.13 0)
     (in_bom yes) (on_board yes) (fields_autoplaced)
-    (property "Reference" "J3" (id 0) (at 154.94 24.1299 0)
+    (property "Reference" "J5" (id 0) (at 154.94 24.1299 0)
       (effects (font (size 1.27 1.27)) (justify left))
     )
@@
   (symbol (lib_id "power:+5VP") (at 76.2 25.4 0) (mirror y)
     (in_bom yes) (on_board yes) (fields_autoplaced)
-    (property "Reference" "#PWR025" (id 0) (at 76.2 29.21 0)
+    (property "Reference" "#PWR037" (id 0) (at 76.2 29.21 0)
       (effects (font (size 1.27 1.27)) hide)
     )
@@
   (symbol (lib_id "power:GND") (at 128.27 88.9 0)
     (in_bom yes) (on_board yes) (fields_autoplaced)
-    (property "Reference" "#PWR027" (id 0) (at 128.27 95.25 0)
+    (property "Reference" "#PWR039" (id 0) (at 128.27 95.25 0)
       (effects (font (size 1.27 1.27)) hide)
     )
@@
   (symbol (lib_id "power:GNDPWR") (at 139.7 34.29 0)
     (in_bom yes) (on_board yes) (fields_autoplaced)
-    (property "Reference" "#PWR028" (id 0) (at 139.7 39.37 0)
-      (effects (font (size 1.27 1.27)) hide)
-    )
+    (property "Reference" "#PWR040" (id 0) (at 139.7 39.37 0)
+      (effects (font (size 1.27 1.27)) hide)
+    )

Commit message: Remove top LED, connect channel LEDs to VIN, expose RX/TX header
Parts:
- R10: renamed from R14; value 470R -> 2kR
- renumbered C6 to C4, D5 to D3, J5 to J3, JP7 to JP3, JP8 to JP4, R13 to R9, U5 to U3
Connections:
- net GND: now also D3.1 (K); no longer R10.1
- net VIN: now also R10.2
- net LED: no longer names the net of D3.2 (A)
- net LED: now also R10.1
Other:
- moved on the sheet: D3, R10
Changed lines of the file:
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@@
-    (stroke (width 0) (type default) (color 0 0 0 0))
-  )
-  (wire (pts (xy 184.15 31.75) (xy 184.15 34.925))
     (stroke (width 0) (type default) (color 0 0 0 0))
   )
@@
     (stroke (width 0) (type default) (color 0 0 0 0))
   )
+  (wire (pts (xy 184.15 44.45) (xy 184.15 48.26))
+    (stroke (width 0) (type default) (color 0 0 0 0))
+  )
   (wire (pts (xy 157.48 87.63) (xy 157.48 80.01))
     (stroke (width 0) (type default) (color 0 0 0 0))
@@
     (stroke (width 0) (type default) (color 0 0 0 0))
   )
-  (wire (pts (xy 184.15 42.545) (xy 184.15 48.26))
-    (stroke (width 0) (type default) (color 0 0 0 0))
-  )
   (wire (pts (xy 138.43 73.66) (xy 146.05 73.66))
     (stroke (width 0) (type default) (color 0 0 0 0))
@@
   )
   (wire (pts (xy 128.27 87.63) (xy 128.27 88.9))
+    (stroke (width 0) (type default) (color 0 0 0 0))
+  )
+  (wire (pts (xy 184.15 31.75) (xy 184.15 36.83))
     (stroke (width 0) (type default) (color 0 0 0 0))
   )
@@
     (effects (font (size 1.27 1.27)) (justify left bottom))
   )
+  (label "VIN" (at 177.8 31.75 0)
+    (effects (font (size 1.27 1.27)) (justify left bottom))
+  )
   (label "VIN" (at 69.85 69.85 180)
     (effects (font (size 1.27 1.27)) (justify right bottom))
@@
     (effects (font (size 1.27 1.27)) (justify left))
   )
-  (hierarchical_label "LED" (shape input) (at 177.8 31.75 180)
-    (effects (font (size 1.27 1.27)) (justify right))
-  )
   (hierarchical_label "A1" (shape passive) (at 146.05 78.74 0)
     (effects (font (size 1.27 1.27)) (justify left))
@@
   (symbol (lib_id "Jumper:Jumper_3_Open") (at 69.85 63.5 0)
     (in_bom yes) (on_board yes)
-    (property "Reference" "JP7" (id 0) (at 69.85 57.15 0))
+    (property "Reference" "JP3" (id 0) (at 69.85 57.15 0))
     (property "Value" "Jumper" (id 1) (at 62.23 67.31 0))
     (property "Footprint" "shared_components:PinHeader_1x03_P2.54mm_Vertical_NoFP" (id 2) (at 69.85 63.5 0)
@@
   (symbol (lib_id "Device:C") (at 157.48 76.2 0)
     (in_bom yes) (on_board yes) (fields_autoplaced)
-    (property "Reference" "C6" (id 0) (at 161.29 74.9299 0)
+    (property "Reference" "C4" (id 0) (at 161.29 74.9299 0)
       (effects (font (size 1.27 1.27)) (justify left))
     )
@@
   (symbol (lib_id "Device:R") (at 113.665 76.2 0)
     (in_bom yes) (on_board yes) (fields_autoplaced)
-    (property "Reference" "R13" (id 0) (at 115.57 74.9299 0)
+    (property "Reference" "R9" (id 0) (at 115.57 74.9299 0)
       (effects (font (size 1.27 1.27)) (justify left))
     )
@@
   (symbol (lib_id "Analog_ADC:INA219AxD") (at 128.27 76.2 0)
     (in_bom yes) (on_board yes) (fields_autoplaced)
-    (property "Reference" "U5" (id 0) (at 130.2894 63.5 0)
+    (property "Reference" "U3" (id 0) (at 130.2894 63.5 0)
       (effects (font (size 1.27 1.27)) (justify left))
     )
@@
     (pin "8")
   )
-  (symbol (lib_id "Device:R") (at 184.15 52.07 180)
-    (in_bom yes) (on_board yes) (fields_autoplaced)
-    (property "Reference" "R14" (id 0) (at 177.8 52.07 90))
-    (property "Value" "470R" (id 1) (at 180.34 52.07 90))
-    (property "Footprint" "Resistor_SMD:R_0805_2012Metric_Pad1.20x1.40mm_HandSolder" (id 2) (at 185.928 52.07 90)
-      (effects (font (size 1.27 1.27)) hide)
-    )
-    (property "Datasheet" "~" (id 3) (at 184.15 52.07 0)
+  (symbol (lib_id "Device:R") (at 184.15 40.64 180)
+    (in_bom yes) (on_board yes) (fields_autoplaced)
+    (property "Reference" "R10" (id 0) (at 177.8 40.64 90))
+    (property "Value" "2kR" (id 1) (at 180.34 40.64 90))
+    (property "Footprint" "Resistor_SMD:R_0805_2012Metric_Pad1.20x1.40mm_HandSolder" (id 2) (at 185.928 40.64 90)
+      (effects (font (size 1.27 1.27)) hide)
+    )
+    (property "Datasheet" "~" (id 3) (at 184.15 40.64 0)
       (effects (font (size 1.27 1.27)) hide)
     )
@@
   (symbol (lib_id "Jumper:Jumper_3_Open") (at 88.9 31.75 0)
     (in_bom yes) (on_board yes)
-    (property "Reference" "JP8" (id 0) (at 88.9 25.4 0))
+    (property "Reference" "JP4" (id 0) (at 88.9 25.4 0))
     (property "Value" "Jumper" (id 1) (at 88.9 38.735 0))
     (property "Footprint" "shared_components:PinHeader_1x03_P2.54mm_Vertical_NoFP" (id 2) (at 88.9 31.75 0)
@@
     (pin "1")
   )
-  (symbol (lib_id "Device:LED") (at 184.15 38.735 90)
-    (in_bom yes) (on_board yes) (fields_autoplaced)
-    (property "Reference" "D5" (id 0) (at 191.77 40.3225 0))
-    (property "Value" "LED" (id 1) (at 189.23 40.3225 0))
-    (property "Footprint" "LED_SMD:LED_1206_3216Metric" (id 2) (at 184.15 38.735 0)
-      (effects (font (size 1.27 1.27)) hide)
-    )
-    (property "Datasheet" "~" (id 3) (at 184.15 38.735 0)
+  (symbol (lib_id "Device:LED") (at 184.15 52.07 90)
+    (in_bom yes) (on_board yes) (fields_autoplaced)
+    (property "Reference" "D3" (id 0) (at 191.77 53.6575 0))
+    (property "Value" "LED" (id 1) (at 189.23 53.6575 0))
+    (property "Footprint" "LED_SMD:LED_1206_3216Metric" (id 2) (at 184.15 52.07 0)
+      (effects (font (size 1.27 1.27)) hide)
+    )
+    (property "Datasheet" "~" (id 3) (at 184.15 52.07 0)
       (effects (font (size 1.27 1.27)) hide)
     )
@@
   (symbol (lib_id "Connector_Generic:Conn_01x04") (at 151.765 24.13 0)
     (in_bom yes) (on_board yes) (fields_autoplaced)
-    (property "Reference" "J5" (id 0) (at 154.94 24.1299 0)
-      (effects (font (size 1.27 1.27)) (justify left))
-    )
+    (property "Reference" "J3" (id 0) (at 154.94 24.1299 0)
+      (effects (font (size 1.27 1.27)) (justify left))
+    )
